File: hw_karifa/karifa.kicad_sch (KiCad schematic)
At the start: 39 parts, among them J1 Conn_2Rows-05Pins, Q1 AO3401A, Q2 AO3401A, Q3 AO3401A, SW1 SW_DPST_x2, T1 Tab, U1 PY32F002AF15P6TU

Commit message: Generalized gitignore + fixed SOT-23 reference
Parts:
- Q1, Q2, Q3: footprint sajat:SOT-23 -> karifa:SOT-23
Changed lines of the file:
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@@
       (effects (font (size 1.27 1.27)))
     )
-    (property "Footprint" "sajat:SOT-23" (at 42.545 67.31 0)
+    (property "Footprint" "karifa:SOT-23" (at 42.545 67.31 0)
       (effects (font (size 1.27 1.27) italic) (justify left) hide)
     )
@@
       (effects (font (size 1.27 1.27)))
     )
-    (property "Footprint" "sajat:SOT-23" (at 42.545 43.18 0)
+    (property "Footprint" "karifa:SOT-23" (at 42.545 43.18 0)
       (effects (font (size 1.27 1.27) italic) (justify left) hide)
     )
@@
       (effects (font (size 1.27 1.27)))
     )
-    (property "Footprint" "sajat:SOT-23" (at 40.005 92.71 0)
+    (property "Footprint" "karifa:SOT-23" (at 40.005 92.71 0)
       (effects (font (size 1.27 1.27) italic) (justify left) hide)
     )
