File: hw_karifa/karifa.kicad_sch (KiCad schematic)
At the start: 39 parts, among them J1 Conn_2Rows-05Pins, Q1 AO3401A, Q2 AO3401A, Q3 AO3401A, SW1 SW_DPST_x2, T1 Tab, U1 PY32F002AF15P6TU

Commit message: Footprint fix for JLCPCB assembly.
Parts:
- D1: footprint LED_SMD:LED_RGB_Wuerth-PLCC4_3.2x2.8mm_150141M173100 -> karifa:LED_RGB_Wuerth-PLCC4_3.2x2.8mm_150141M173100
- U1: footprint Package_SO:TSSOP-20_4.4x6.5mm_P0.65mm -> karifa:TSSOP-20_4.4x6.5mm_P0.65mm
Changed lines of the file:
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@@
       (effects (font (size 1.27 1.27)))
     )
-    (property "Footprint" "Package_SO:TSSOP-20_4.4x6.5mm_P0.65mm" (at 187.96 104.14 0)
+    (property "Footprint" "karifa:TSSOP-20_4.4x6.5mm_P0.65mm" (at 187.96 104.14 0)
       (effects (font (size 1.27 1.27)) hide)
     )
@@
       (effects (font (size 1.27 1.27)) (justify left))
     )
-    (property "Footprint" "LED_SMD:LED_RGB_Wuerth-PLCC4_3.2x2.8mm_150141M173100" (at 66.04 101.6 0)
-      (effects (font (size 1.27 1.27)) hide)
-    )
+    (property "Footprint" "karifa:LED_RGB_Wuerth-PLCC4_3.2x2.8mm_150141M173100" (at 66.04 101.6 0)
+      (effects (font (size 1.27 1.27)) hide)
+    )
