File: hw_box/panel.kicad_pcb (KiCad board)
At the start: 2 copper layers, 111.5 x 173.3 mm, 284 parts, among them J1 Conn_2Rows-05Pins, SW1 SW_DPST_x2, U1 PY32F002AF15P6TU

Commit message: box Rev.B
modified the F. Mask, and rotate the Led4 and Led12
Parts:
- removed the C1 at (120.2, 157.5)
- removed the C1 at (120.2, 49.3)
- removed the C1 at (120.2, 103.4)
- removed the C1 at (169.5, 157.5)
- removed the C1 at (169.5, 49.3)
- removed the C1 at (169.5, 103.4)
- removed the C2 at (173.2, 126.0)
- removed the C2 at (173.2, 71.9)
- removed the C2 at (124.0, 180.1)
- removed the C2 at (124.0, 126.0)
- removed the C2 at (124.0, 71.9)
- removed the C2 at (173.2, 180.1)
- added C1: 100nF, Capacitor_SMD:C_0805_2012Metric, F.Cu at (173.2, 126.0)
- added C1: 100nF, Capacitor_SMD:C_0805_2012Metric, F.Cu at (124.0, 126.0)
- added C1: 100nF, Capacitor_SMD:C_0805_2012Metric, F.Cu at (173.2, 71.9)
- added C1: 100nF, Capacitor_SMD:C_0805_2012Metric, F.Cu at (173.2, 180.1)
- added C1: 100nF, Capacitor_SMD:C_0805_2012Metric, F.Cu at (124.0, 71.9)
- added C1: 100nF, Capacitor_SMD:C_0805_2012Metric, F.Cu at (124.0, 180.1)
- added C2: 10uF, Capacitor_SMD:C_0805_2012Metric, F.Cu at (169.5, 49.3)
- added C2: 10uF, Capacitor_SMD:C_0805_2012Metric, F.Cu at (169.5, 157.5)
- added C2: 10uF, Capacitor_SMD:C_0805_2012Metric, F.Cu at (120.2, 157.5)
- added C2: 10uF, Capacitor_SMD:C_0805_2012Metric, F.Cu at (169.5, 103.4)
- added C2: 10uF, Capacitor_SMD:C_0805_2012Metric, F.Cu at (120.2, 103.4)
- added C2: 10uF, Capacitor_SMD:C_0805_2012Metric, F.Cu at (120.2, 49.3)
- turned D12 to 26.566 degrees (x6)
- turned D4 to 153.436 degrees (x6)
Routing:
- net Board_3-GND: track 64.9 -> 0.07 mm
- net Board_2-GND: track 64.9 -> 0.07 mm
- net Board_1-GND: track 64.9 -> 0.07 mm
- net Board_5-GND: track 64.9 -> 0.07 mm
- net Board_4-GND: track 64.9 -> 0.07 mm
- net Board_0-GND: track 64.9 -> 0.07 mm
- net Board_4-Net-(D12-A): track 9.26 -> 27.1 mm, vias 0 -> 3
- net Board_2-Net-(D12-A): track 9.26 -> 27.1 mm, vias 0 -> 3
- net Board_0-Net-(D12-A): track 9.26 -> 27.1 mm, vias 0 -> 3
- net Board_5-Net-(D12-A): track 9.26 -> 27.1 mm, vias 0 -> 3
- net Board_1-Net-(D12-A): track 9.26 -> 27.1 mm, vias 0 -> 3
- net Board_3-Net-(D12-A): track 9.26 -> 27.1 mm, vias 0 -> 3
- net Board_3-/MPX2: track 132.0 -> 116.0 mm, vias 9 -> 12
- net Board_4-/MPX2: track 132.0 -> 116.0 mm, vias 9 -> 12
- net Board_2-/MPX2: track 132.0 -> 116.0 mm, vias 9 -> 12
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Other:
- outline, holes or cut-outs redrawn
- board text added: "Rev. B"
- board text removed: "Rev. A"
