File: hw_macskas/macskas.kicad_pcb (KiCad board)
At the start: 2 copper layers, 49 x 54.5 mm, 44 parts, among them J1 Conn_2Rows-05Pins, Q1 AO3401A, Q2 AO3401A, Q3 AO3401A, SW1 SW_DPST_x2, T1 Tab, U1 PY32F002AF15P6TU

Commit message: Working on cat design.
Parts:
- removed D1: LED_ARGB, karifa:LED_RGB_Wuerth-PLCC4_3.2x2.8mm_150141M173100
- removed D10, D11, D12, D13, D2, D3, D4, D5, D6, D7, D8, D9: LED, LED_SMD:LED_0805_2012Metric
- removed R11, R12: 100k, Resistor_SMD:R_0603_1608Metric
- BT1: value Battery -> CR2032
- C1: value 100nF -> 10uF
- C3: value 10uF -> 100nF
- L1, L2, L3: value L -> 1mH; footprint Inductor_SMD:L_1008_2520Metric -> Inductor_SMD:L_Ferrocore_DLG-0403
- R2, R3: value 100k -> 1k
- R8, R9: value 1k -> 100k
- moved C1 65.6 mm to (132.8, 101.9)
- moved R3 61.3 mm to (143.3, 99.1), turned to 180 degrees
- moved Q3 59.3 mm to (133.2, 73.8)
- moved R1 58.6 mm to (131.2, 56.0)
- moved R9 54.5 mm to (129.3, 96.1), turned to 180 degrees
- moved J1 53.4 mm to (127.9, 91.5)
- moved U1 53.4 mm to (136.2, 97.0)
- moved C2 53.3 mm to (139.6, 101.9)
- moved R2 53.1 mm to (143.3, 100.9), turned to 180 degrees
- moved Q1 52.1 mm to (135.2, 56.5)
- moved R4 51.7 mm to (143.3, 97.4)
- moved R5 51.7 mm to (143.3, 95.6)
- moved R6 51.7 mm to (143.3, 93.9)
- moved R7 51.7 mm to (143.3, 92.1)
- moved L1 50.7 mm to (141.0, 56.8)
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- renumbered T1 to T2, T1 to T3, T1 to T4, T1 to T5, T1 to T6
Connections:
- C1 pad 1: GND -> VCC
- C1 pad 2: VCC -> GND
- C3 pad 1: VCC -> GND
- C3 pad 2: GND -> VCC
- L1 pad 2: GND -> /MPX1
- L2 pad 2: GND -> /MPX2
- Q1 pad 1: /B -> /MPX1
- Q2 pad 1: /R -> /MPX2
- Q3 pad 1: /G -> /MPX3
- R1 pad 2: /B -> /MPX1
- R10 pad 2: /nRST -> /MPX3
- R2 pad 1: VCC -> Net-(D1-A)
- R2 pad 2: /R -> /L1
- R3 pad 1: VCC -> Net-(D14-A)
- R3 pad 2: /G -> /L2
- R4 pad 2: /L1 -> /L3
- R5 pad 2: /L2 -> /L4
- R6 pad 2: /L3 -> /L5
- R7 pad 2: /L4 -> /L6
- R8 pad 1: Net-(D10-A) (its old number) -> VCC
- R8 pad 2: /L5 -> /MPX2
- R9 pad 1: Net-(D12-A) (its old number) -> Net-(SW1A-A)
- R9 pad 2: /L6 -> VCC
- U1 pad 11: /R -> /MPX2
- U1 pad 12: /B -> /MPX1
- U1 pad 14: /G -> /MPX3
- U1 pad 5: Net-(U1-PB6/PF4-BOOT0) -> unconnected-(U1-PB6/PF4-BOOT0-Pad5)
- U1 pad 6: /MPX1 -> unconnected-(U1-PA6-Pad6)
- U1 pad 7: /MPX2 -> unconnected-(U1-PA5-Pad7)
Other:
- board size 49 x 54.5 mm -> 49 x 59.5 mm

Commit message: Updated cat.
Parts:
- added D1: LED, LED_SMD:LED_0805_2012Metric, F.Cu at (123.0, 100.0)
- added D10: LED, LED_SMD:LED_0805_2012Metric, F.Cu at (78.4, 107.9)
- added D11: LED, LED_SMD:LED_0805_2012Metric, F.Cu at (96.0, 122.7)
- added D12: LED, LED_SMD:LED_0805_2012Metric, F.Cu at (117.6, 114.8)
- added D13: LED, LED_SMD:LED_0805_2012Metric, F.Cu at (117.6, 85.2)
- added D14: LED, LED_SMD:LED_0805_2012Metric, F.Cu at (96.0, 77.3)
- added D15: LED, LED_SMD:LED_0805_2012Metric, F.Cu at (78.4, 92.1)
- added D16: LED, LED_SMD:LED_0805_2012Metric, F.Cu at (82.4, 114.8)
- added D17: LED, LED_SMD:LED_0805_2012Metric, F.Cu at (104.0, 122.7)
- added D18: LED, LED_SMD:LED_0805_2012Metric, F.Cu at (121.6, 107.9)
- added D2: LED, LED_SMD:LED_0805_2012Metric, F.Cu at (111.5, 80.1)
- added D3: LED, LED_SMD:LED_0805_2012Metric, F.Cu at (88.5, 80.1)
- added D4: LED, LED_SMD:LED_0805_2012Metric, F.Cu at (77.0, 100.0)
- added D5: LED, LED_SMD:LED_0805_2012Metric, F.Cu at (88.5, 119.9)
- added D6: LED, LED_SMD:LED_0805_2012Metric, F.Cu at (111.5, 119.9)
- added D7: LED, LED_SMD:LED_0805_2012Metric, F.Cu at (121.6, 92.1)
- added D8: LED, LED_SMD:LED_0805_2012Metric, F.Cu at (104.0, 77.3)
- added D9: LED, LED_SMD:LED_0805_2012Metric, F.Cu at (82.4, 85.2)
- R2, R3, R4, R5, R6, R7: value 1k -> 10
- moved SW1 94.9 mm to (96.5, 82.5)
- moved BT1 86.6 mm to (99.8, 87.7), turned to -90 degrees
- moved L2 64.7 mm to (85.2, 95.5), turned to 0 degrees
- moved Q2 57.3 mm to (84.2, 91.0), turned to 0 degrees
- moved R8 56.2 mm to (87.2, 91.0), turned to -90 degrees
- moved L3 53.7 mm to (107.5, 116.0), turned to 90 degrees
- moved Q3 52.8 mm to (103.0, 117.0)
- moved R10 52.8 mm to (103.0, 114.0)
- moved R1 43.0 mm to (114.8, 95.8), turned to 90 degrees
- moved Q1 42.9 mm to (117.8, 95.8), turned to 180 degrees
- moved U1 42.5 mm to (93.8, 95.8)
- moved L1 42.1 mm to (116.8, 91.2), turned to 180 degrees
- moved R2 42.1 mm to (101.2, 101.8)
- moved R3 42.1 mm to (101.2, 100.0)
- moved R4 42.1 mm to (101.2, 98.2)
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Connections:
- L3 pad 2: GND -> /MPX3
Other:
- board text removed: "PCB by Kristóf"

Commit message: Macskas routed.
Parts:
- moved C2 3.25 mm to (101.2, 112.0), turned to 180 degrees
Routing:
- net Net-(D10-K): track 0.00 -> 141.2 mm, vias 0 -> 7
- net Net-(D13-K): track 0.00 -> 133.8 mm, vias 0 -> 7
- net Net-(D1-K): track 0.00 -> 124.5 mm, vias 0 -> 2
- net VCC: track 0.00 -> 82.4 mm, vias 0 -> 1
- net Net-(D10-A): track 0.00 -> 58.1 mm, vias 0 -> 2
- net Net-(D11-A): track 0.00 -> 56.8 mm
- net Net-(D15-A): track 0.00 -> 49.3 mm, vias 0 -> 2
- net GND: track 0.00 -> 47.9 mm, vias 0 -> 53
- net Net-(D12-A): track 0.00 -> 46.0 mm
- net Net-(D1-A): track 0.00 -> 40.3 mm, vias 0 -> 2
- net Net-(D14-A): track 0.00 -> 40.3 mm, vias 0 -> 2
- net /MPX3: track 0.00 -> 32.5 mm, vias 0 -> 2
- net /MPX1: track 0.00 -> 28.7 mm, vias 0 -> 2
- net /nRST: track 0.00 -> 27.5 mm, vias 0 -> 1
- net /MPX2: track 0.00 -> 20.8 mm, vias 0 -> 2
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- added copper zone on B.Cu, net GND
- added copper zone on F.Cu, net GND

Commit message: Panelized.
Parts:
- removed T4, T5, T6: Tab, kikit:Tab
- T1, T2, T3: footprint kikit:Tab -> PCM_kikit:Tab
- moved T3 155.8 mm to (71.9, 100.0), turned to 0 degrees
- moved T1 123.2 mm to (100.0, 126.6), turned to 90 degrees
- moved T2 106.3 mm to (126.7, 100.0)

Commit message: Soldering guide.
Parts:
- D1, D2, D3, D4, D5, D6: value LED -> Green
- D10, D11, D12, D7, D8, D9: value LED -> White
- D13, D14, D15, D16, D17, D18: value LED -> Red
Changed lines of the file:
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@@
 			)
 		)
-		(property "Value" "LED"
+		(property "Value" "White"
 			(at 0 1.65 110)
 			(layer "F.Fab")
@@
 			(at 0 3.2 0)
 			(layer "F.Fab")
+			(hide yes)
 			(effects
 				(font
@@
 			)
 		)
-		(property "Value" "LED"
+		(property "Value" "Red"
 			(at 0.000001 1.65 130)
 			(layer "F.Fab")
@@
 			(at 0 1.43 90)
 			(layer "F.Fab")
+			(hide yes)
 			(effects
 				(font
@@
 			(at 0 1.43 0)
 			(layer "F.Fab")
+			(hide yes)
 			(effects
 				(font
@@
 			)
 		)
-		(property "Value" "LED"
+		(property "Value" "Green"
 			(at 0 1.65 150)
 			(layer "F.Fab")
@@
 			(at 0.439 1.43 90)
 			(layer "F.Fab")
+			(hide yes)
 			(effects
 				(font
@@
 			)
 		)
-		(property "Value" "LED"
+		(property "Value" "White"
 			(at 0.000001 1.65 170)
 			(layer "F.Fab")
@@
 			(at 0 -2.4 90)
 			(layer "F.Fab")
+			(hide yes)
 			(effects
 				(font
@@
 		)
 		(fp_text user "${REFERENCE}"
-			(at 0 0 90)
+			(at 0 0 180)
 			(layer "F.Fab")
 			(effects
@@
 			(at 0.635 4.235 0)
 			(layer "F.Fab")
+			(hide yes)
 			(effects
 				(font
@@
 		)
 		(fp_text user "${REFERENCE}"
-			(at 0.635 1.27 90)
+			(at 0.625 0.79 180)
 			(layer "F.Fab")
 			(effects
@@
 			)
 		)
-		(property "Value" "LED"
+		(property "Value" "Red"
 			(at -0.000001 1.65 10)
 			(layer "F.Fab")
@@
 			(at 0 3.2 0)
 			(layer "F.Fab")
+			(hide yes)
 			(effects
 				(font
@@
 			(at 0 1.43 0)
 			(layer "F.Fab")
+			(hide yes)
 			(effects
 				(font
@@
 			)
 		)
-		(property "Value" "LED"
+		(property "Value" "Green"
 			(at 0 1.65 90)
 			(layer "F.Fab")
@@
 			)
 		)
-		(property "Value" "LED"
+		(property "Value" "Green"
 			(at 0 1.65 90)
 			(layer "F.Fab")
@@
 			)
 		)
-		(property "Value" "LED"
+		(property "Value" "Red"
 			(at -0.000001 1.65 10)
 			(layer "F.Fab")
@@
 			(at 0 -2.4 0)
 			(layer "F.Fab")
+			(hide yes)
 			(effects
 				(font
@@
 		)
 		(fp_text user "${REFERENCE}"
-			(at 0 0 0)
+			(at 0 0 90)
 			(layer "F.Fab")
 			(effects
@@
 			)
 		)
-		(property "Value" "LED"
+		(property "Value" "White"
 			(at -0.000001 1.65 50)
 			(layer "F.Fab")
@@
 			(at 0 4.199999 0)
 			(layer "F.Fab")
+			(hide yes)
 			(effects
 				(font
@@
 			(at 0 3.75 0)
 			(layer "F.Fab")
+			(hide yes)
 			(effects
 				(font
@@
 		)
 		(fp_text user "${REFERENCE}"
-			(at 0 -3.75 0)
+			(at -4.4 0 0)
 			(layer "F.Fab")
 			(effects
@@
 			(at 0 1.43 0)
 			(layer "F.Fab")
+			(hide yes)
 			(effects
 				(font
@@
 			(at 0 1.43 0)
 			(layer "F.Fab")
+			(hide yes)
 			(effects
 				(font
@@
 			)
 		)
-		(property "Value" "LED"
+		(property "Value" "Green"
 			(at 0 1.65 30)
 			(layer "F.Fab")
@@
 			)
 		)
-		(property "Value" "LED"
+		(property "Value" "Red"
 			(at 0 1.65 70)
 			(layer "F.Fab")
@@
 			(at 0 1.68 0)
 			(layer "F.Fab")
+			(hide yes)
 			(effects
 				(font
@@
 			)
 		)
-		(property "Value" "LED"
+		(property "Value" "Red"
 			(at 0.000001 1.65 130)
 			(layer "F.Fab")
@@
 			(at 0 1.68 0)
 			(layer "F.Fab")
+			(hide yes)
 			(effects
 				(font
@@
 			(at 0 1.679999 0)
 			(layer "F.Fab")
+			(hide yes)
 			(effects
 				(font
@@
 			(at 0 1.43 0)
 			(layer "F.Fab")
+			(hide yes)
 			(effects
 				(font
@@
 			(at 0 -2.4 0)
 			(layer "F.Fab")
+			(hide yes)
 			(effects
 				(font
@@
 		)
 		(fp_text user "${REFERENCE}"
-			(at 0 0 0)
+			(at 0 0 90)
 			(layer "F.Fab")
 			(effects
@@
 			)
 		)
-		(property "Value" "LED"
+		(property "Value" "White"
 			(at 0.000001 1.65 170)
 			(layer "F.Fab")
@@
 			(at 0 1.43 0)
 			(layer "F.Fab")
+			(hide yes)
 			(effects
 				(font
@@
 			)
 		)
-		(property "Value" "LED"
+		(property "Value" "White"
 			(at -0.000001 1.65 50)
 			(layer "F.Fab")
@@
 			(at 0 1.43 0)
 			(layer "F.Fab")
+			(hide yes)
 			(effects
 				(font
@@
 			(at 0 3.2 90)
 			(layer "F.Fab")
+			(hide yes)
 			(effects
 				(font
@@
 			)
 		)
-		(property "Value" "LED"
+		(property "Value" "Green"
 			(at 0 1.65 150)
 			(layer "F.Fab")
@@
 			)
 		)
-		(property "Value" "LED"
+		(property "Value" "Red"
 			(at 0 1.65 70)
 			(layer "F.Fab")
@@
 			)
 		)
-		(property "Value" "LED"
+		(property "Value" "Green"
 			(at 0 1.65 30)
 			(layer "F.Fab")
@@
 			(at 0 1.43 0)
 			(layer "F.Fab")
+			(hide yes)
 			(effects
 				(font
@@
 			)
 		)
-		(property "Value" "LED"
+		(property "Value" "White"
 			(at 0 1.65 110)
 			(layer "F.Fab")
