File: hw_angyalka/angyalka.kicad_sch (KiCad schematic)
At the start: 34 parts, among them J1 Conn_2Rows-05Pins, Q1 AO3401A, Q2 AO3401A, SW1 SW_DPST_x2, T1 Tab, T2 Tab, T3 Tab, U1 PY32F002AF15P6TU

Commit message: Fixed LED resistors.
Parts:
- R2, R3, R4, R5, R6, R7: value 1k -> 10
Changed lines of the file:
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@@
 		(dnp no)
 		(property "Reference" "R7"
-			(at 246.38 91.694 90)
-			(effects
-				(font
-					(size 1.27 1.27)
-				)
-				(justify left)
-			)
-		)
-		(property "Value" "1k"
+			(at 243.84 86.614 90)
+			(effects
+				(font
+					(size 1.27 1.27)
+				)
+				(justify left)
+			)
+		)
+		(property "Value" "10"
 			(at 243.84 91.694 90)
 			(effects
@@
 		(dnp no)
 		(property "Reference" "R4"
-			(at 189.23 91.694 90)
-			(effects
-				(font
-					(size 1.27 1.27)
-				)
-				(justify left)
-			)
-		)
-		(property "Value" "1k"
+			(at 186.69 86.614 90)
+			(effects
+				(font
+					(size 1.27 1.27)
+				)
+				(justify left)
+			)
+		)
+		(property "Value" "10"
 			(at 186.69 91.694 90)
 			(effects
@@
 		(dnp no)
 		(property "Reference" "R2"
-			(at 151.13 91.694 90)
-			(effects
-				(font
-					(size 1.27 1.27)
-				)
-				(justify left)
-			)
-		)
-		(property "Value" "1k"
+			(at 148.336 86.868 90)
+			(effects
+				(font
+					(size 1.27 1.27)
+				)
+				(justify left)
+			)
+		)
+		(property "Value" "10"
 			(at 148.59 91.694 90)
 			(effects
@@
 		(dnp no)
 		(property "Reference" "R3"
-			(at 170.18 91.44 90)
-			(effects
-				(font
-					(size 1.27 1.27)
-				)
-				(justify left)
-			)
-		)
-		(property "Value" "1k"
+			(at 167.64 86.614 90)
+			(effects
+				(font
+					(size 1.27 1.27)
+				)
+				(justify left)
+			)
+		)
+		(property "Value" "10"
 			(at 167.64 91.44 90)
 			(effects
@@
 		(dnp no)
 		(property "Reference" "R6"
-			(at 227.33 91.694 90)
-			(effects
-				(font
-					(size 1.27 1.27)
-				)
-				(justify left)
-			)
-		)
-		(property "Value" "1k"
+			(at 224.536 86.36 90)
+			(effects
+				(font
+					(size 1.27 1.27)
+				)
+				(justify left)
+			)
+		)
+		(property "Value" "10"
 			(at 224.79 91.694 90)
 			(effects
@@
 		(dnp no)
 		(property "Reference" "R5"
-			(at 208.28 91.694 90)
-			(effects
-				(font
-					(size 1.27 1.27)
-				)
-				(justify left)
-			)
-		)
-		(property "Value" "1k"
+			(at 205.74 86.614 90)
+			(effects
+				(font
+					(size 1.27 1.27)
+				)
+				(justify left)
+			)
+		)
+		(property "Value" "10"
 			(at 205.74 91.694 90)
 			(effects
