File: hw_angyalka/angyalka.kicad_pcb (KiCad board)
At the start: 2 copper layers, 82.9 x 59.5 mm, 34 parts, among them J1 Conn_2Rows-05Pins, Q1 AO3401A, Q2 AO3401A, SW1 SW_DPST_x2, T1 Tab, T2 Tab, T3 Tab, U1 PY32F002AF15P6TU

Commit message: Covered F.Mask around soldering pads
Parts:
- moved D7 0.60 mm to (148.5, 127.4)
- moved D2 0.58 mm to (164.7, 123.5)
- moved D8 0.42 mm to (132.3, 123.7)
Routing:
- net Net-(D1-K): track 8.21 -> 5.52 mm
- net Net-(D10-K): track 17.5 -> 16.9 mm
- net Net-(D1-A): track 17.0 -> 16.4 mm
- removed copper zone on B.Cu, net (none)

Commit message: Angyalka panelized.
Parts:
- moved T2 145.9 mm to (173.9, 115.0), turned to 180 degrees
- moved T3 132.5 mm to (148.2, 135.9)
- moved T1 71.8 mm to (124.5, 115.0)
Other:
- board text added: "Rev.A"
- board text removed: "Every machine is a smoke machine if you operate it wrong enough."
- board text removed: "Rev.B"
Changed lines of the file:
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@@
 	(footprint "PCM_kikit:Tab"
 		(layer "F.Cu")
-		(at 51.75 35.24159 -90)
+		(at 173.9 115 180)
 		(descr "A symbol representing annotation for tab placement")
 		(property "Reference" "T2"
-			(at -0.25 -2 270)
+			(at -0.25 -2 0)
 			(layer "F.SilkS")
 			(hide yes)
@@
 		)
 		(property "Value" "Tab"
-			(at -3 -1 270)
+			(at -3 -1 0)
 			(layer "Dwgs.User")
 			(effects
@@
 		)
 		(property "Datasheet" ""
-			(at 0 0 270)
+			(at 0 0 0)
 			(layer "F.Fab")
 			(hide yes)
@@
 		)
 		(property "Description" ""
-			(at 0 0 270)
+			(at 0 0 0)
 			(layer "F.Fab")
 			(hide yes)
@@
 		(fp_line
 			(start 0 0)
-			(end -3 0)
+			(end -1 -1)
 			(stroke
 				(width 0.3)
@@
 		(fp_line
 			(start 0 0)
-			(end -1 -1)
+			(end -3 0)
 			(stroke
 				(width 0.3)
@@
 		)
 		(fp_text user "KIKIT: width: 3mm"
-			(at -5.5 0 0)
+			(at -5.5 0 90)
 			(layer "Dwgs.User")
 			(effects
@@
 	(footprint "PCM_kikit:Tab"
 		(layer "F.Cu")
-		(at 66.5 72.75)
+		(at 124.5 115)
 		(descr "A symbol representing annotation for tab placement")
 		(property "Reference" "T1"
@@
 	(footprint "PCM_kikit:Tab"
 		(layer "F.Cu")
-		(at 53.75 43.05 90)
+		(at 148.25 135.95 90)
 		(descr "A symbol representing annotation for tab placement")
 		(property "Reference" "T3"
@@
 	)
 	(gr_arc
-		(start 145.115185 76.81047)
+		(start 145.115249 76.810441)
 		(mid 148.427731 75.999829)
-		(end 151.76802 76.687267)
+		(end 151.76803 76.687217)
 		(stroke
 			(width 0.1)
-			(type default)
+			(type solid)
 		)
 		(layer "Edge.Cuts")
@@
 	)
 	(gr_arc
-		(start 152.646715 75.511847)
-		(mid 152.739342 76.497246)
-		(end 151.76802 76.68731)
+		(start 144.356687 75.576441)
+		(mid 148.487794 73.800006)
+		(end 152.646687 75.510241)
 		(stroke
 			(width 0.1)
-			(type default)
+			(type solid)
 		)
 		(layer "Edge.Cuts")
 	)
 	(gr_arc
-		(start 144.356719 75.576407)
-		(mid 148.487794 73.800006)
-		(end 152.646715 75.51021)
+		(start 145.115249 76.810441)
+		(mid 144.225577 76.506048)
+		(end 144.356687 75.576441)
 		(stroke
 			(width 0.1)
-			(type default)
+			(type solid)
 		)
 		(layer "Edge.Cuts")
 	)
 	(gr_arc
-		(start 145.115185 76.81047)
-		(mid 144.225577 76.506048)
-		(end 144.358116 75.575184)
+		(start 152.646687 75.510241)
+		(mid 152.739342 76.497204)
+		(end 151.76803 76.687217)
 		(stroke
 			(width 0.1)
-			(type default)
+			(type solid)
 		)
 		(layer "Edge.Cuts")
 	)
-	(gr_text "Rev.B"
+	(gr_text "Rev.A"
 		(at 143 118.5 90)
 		(layer "B.SilkS")
@@
 		(layer "B.SilkS")
 		(effects
-			(font
-				(size 1 1)
-				(thickness 0.15)
-			)
-			(justify left bottom mirror)
-		)
-	)
-	(gr_text "Every machine is a\nsmoke machine if\nyou operate it \nwrong enough."
-		(at 212 119.75 0)
-		(layer "B.SilkS")
-		(effects

Commit message: Updated value fields.
Parts:
- R2, R3, R4, R5, R6, R7: value 1k -> 10
Changed lines of the file:
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@@
 			)
 		)
-		(property "Value" "1k"
+		(property "Value" "10"
 			(at 0 1.43 0)
 			(layer "F.Fab")
@@
 			)
 		)
-		(property "Value" "1k"
+		(property "Value" "10"
 			(at 0 1.43 0)
 			(layer "F.Fab")
@@
 			)
 		)
-		(property "Value" "1k"
+		(property "Value" "10"
 			(at 0 1.43 0)
 			(layer "F.Fab")
@@
 			)
 		)
-		(property "Value" "1k"
+		(property "Value" "10"
 			(at 0 1.43 0)
 			(layer "F.Fab")
@@
 			)
 		)
-		(property "Value" "1k"
+		(property "Value" "10"
 			(at 0 1.43 0)
 			(layer "F.Fab")
@@
 			)
 		)
-		(property "Value" "1k"
+		(property "Value" "10"
 			(at 0 1.43 0)
 			(layer "F.Fab")
