File: hw_hullocsillag/hullocsillag.kicad_pcb (KiCad board)
At the start: 2 copper layers, 110 x 56 mm, 34 parts, among them J1 Conn_2Rows-05Pins, Q1 AO3401A, Q2 AO3401A, SW1 SW_DPST_x2, T1 Tab, T2 Tab, T3 Tab, U1 PY32F002AF15P6TU

Commit message: Updated value fields.
Parts:
- R2, R3, R4, R5, R6, R7: value 1k -> 10
Changed lines of the file:
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@@
 			)
 		)
-		(property "Value" "1k"
+		(property "Value" "10"
 			(at 0 1.43 0)
 			(layer "F.Fab")
@@
 			)
 		)
-		(property "Value" "1k"
+		(property "Value" "10"
 			(at 0 1.43 0)
 			(layer "F.Fab")
@@
 			)
 		)
-		(property "Value" "1k"
+		(property "Value" "10"
 			(at 0 1.43 164)
 			(layer "F.Fab")
@@
 		(fp_line
 			(start -1.685 0.96)
-			(end 1 0.959997)
+			(end 1 0.959996)
 			(stroke
 				(width 0.12)
@@
 			)
 		)
-		(property "Value" "1k"
+		(property "Value" "10"
 			(at 0 1.43 0)
 			(layer "F.Fab")
@@
 			)
 		)
-		(property "Value" "1k"
+		(property "Value" "10"
 			(at 0 1.43 174)
 			(layer "F.Fab")
@@
 			)
 		)
-		(property "Value" "1k"
+		(property "Value" "10"
 			(at 0 1.43 159)
 			(layer "F.Fab")
